File: PCBs/Driver Carrier v1/Driver Carrier v1.kicad_pcb (KiCad board)
At the start: 2 copper layers, 36 parts, among them J1 Conn_01x08_Socket, J10 Conn_01x08_Socket, J11 Conn_01x04_Pin, J12 Conn_01x08_Socket, J13 Conn_01x08_Socket, J14 Conn_01x04_Pin, J15 Conn_01x08_Socket, J16 Conn_01x08_Socket, J17 Conn_01x04_Pin, J18 Conn_01x08_Socket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

Commit message: Continued working on the PCB
Parts:
- removed J1, J12, J13, J15, J16, J18, J2: Conn_01x08_Socket, Connector_PinSocket_2.54mm:PinSocket_1x08_P2.54mm_Vertical
- removed J14, J17, J29, J5: Conn_01x04_Pin, Connector_PinHeader_2.54mm:PinHeader_1x04_P2.54mm_Vertical
- removed J28: Ground Connectors, Connector_PinHeader_2.54mm:PinHeader_1x02_P2.54mm_Vertical
- removed U1: ESP32-S3-DevKitC, Custom_Footprints:ESP32-S3-DEVKITC Female Headers
- added U10: SILENTSTEPSTICK TMC5160, Custom_Footprints:SILENTSTEPSTICK TMC5160, B.Cu at (63.5, 104.8)
- added U11: SILENTSTEPSTICK TMC2130, Custom_Footprints:SILENTSTEPSTICK TMC2130, B.Cu at (63.5, 100.3)
- added U12: SILENTSTEPSTICK TMC5160, Custom_Footprints:SILENTSTEPSTICK TMC5160, B.Cu at (142.2, 132.1)
- added U13: SILENTSTEPSTICK TMC2130, Custom_Footprints:SILENTSTEPSTICK TMC2130, B.Cu at (142.2, 136.5)
- added U14: SILENTSTEPSTICK TMC5160, Custom_Footprints:SILENTSTEPSTICK TMC5160, B.Cu at (142.2, 100.3)
- added U15: SILENTSTEPSTICK TMC2130, Custom_Footprints:SILENTSTEPSTICK TMC2130, B.Cu at (142.2, 104.8)
- added U16: SILENTSTEPSTICK TMC5160, Custom_Footprints:SILENTSTEPSTICK TMC5160, B.Cu at (63.5, 136.5)
- added U17: SILENTSTEPSTICK TMC2130, Custom_Footprints:SILENTSTEPSTICK TMC2130, B.Cu at (63.5, 132.1)
- added U18: SILENTSTEPSTICK TMC5160, Custom_Footprints:SILENTSTEPSTICK TMC5160, B.Cu at (142.2, 68.6)
- added U19: SILENTSTEPSTICK TMC2130, Custom_Footprints:SILENTSTEPSTICK TMC2130, B.Cu at (142.2, 73.0)
- added U3: ESP32-S3-DEVKITM, Custom_Footprints:ESP32-S3-DEVKITM Female Headers, F.Cu at (90.0, 144.2)
- added U8: SILENTSTEPSTICK TMC5160, Custom_Footprints:SILENTSTEPSTICK TMC5160, B.Cu at (63.5, 73.0)
- added U9: SILENTSTEPSTICK TMC2130, Custom_Footprints:SILENTSTEPSTICK TMC2130, B.Cu at (63.5, 68.6)
- J10, J6, J7, J9: value Conn_01x08_Socket -> Conn_01x04_Pin; footprint Connector_PinSocket_2.54mm:PinSocket_1x08_P2.54mm_Vertical -> Connector_PinHeader_2.54mm:PinHeader_1x04_P2.54mm_Vertical
- J4: value Conn_01x08_Socket -> Screw_Terminal_01x02; footprint Connector_PinSocket_2.54mm:PinSocket_1x08_P2.54mm_Vertical -> Custom_Footprints:Phoenix_TerminalBlock_1x02_3.5mm_1984617
- moved J22 114.6 mm to (148.6, 118.7), turned to -90 degrees
- moved J11 106.8 mm to (147.3, 74.3), turned to 180 degrees
- moved J8 95.3 mm to (147.3, 137.8), turned to 180 degrees
- moved J21 89.9 mm to (57.1, 118.7), turned to 90 degrees
- moved J23 88.6 mm to (148.6, 87.0), turned to -90 degrees
- moved C4 77.9 mm to (123.2, 118.7)
- moved J9 72.4 mm to (147.3, 106.0), turned to 180 degrees
- moved J24 67.4 mm to (148.6, 53.3), turned to -90 degrees
- moved C1 65.6 mm to (82.5, 55.2), turned to 180 degrees
- moved C5 64.7 mm to (123.2, 87.0)
- moved J20 57.9 mm to (57.1, 87.0), turned to 90 degrees
- moved J7 56.0 mm to (58.4, 99.1)
- moved C3 53.4 mm to (82.5, 118.7), turned to 180 degrees
- moved J27 49.9 mm to (106.0, 70.5), turned to 90 degrees
- moved J25 48.6 mm to (99.7, 70.5), turned to -90 degrees
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Connections:
- J10 pad 1: GND -> /All TMCs/BothTMCs n3/M2B
- J10 pad 2: VIO -> /All TMCs/BothTMCs n3/M2A
- J10 pad 3: M1B -> /All TMCs/BothTMCs n3/M1A
- J10 pad 4: M1A -> /All TMCs/BothTMCs n3/M1B
- J11 pad 1: M2B -> /All TMCs/BothTMCs n6/M2B
- J11 pad 2: M2A -> /All TMCs/BothTMCs n6/M2A
- J11 pad 3: M1A -> /All TMCs/BothTMCs n6/M1A
- J11 pad 4: M1B -> /All TMCs/BothTMCs n6/M1B
- J19 pad 1: GND -> SW1
- J19 pad 2: SW1 -> GND
- J19 pad 3: unconnected-(J19-Pin_3-Pad3) -> GND
- J20 pad 1: GND -> SW2
- J20 pad 2: SW2 -> GND
- J20 pad 3: unconnected-(J20-Pin_3-Pad3) -> GND
- J21 pad 1: GND -> SW3
- J21 pad 2: SW3 -> GND
- J21 pad 3: unconnected-(J21-Pin_3-Pad3) -> GND
- J22 pad 1: GND -> SW4
- J22 pad 2: SW4 -> GND
- J22 pad 3: unconnected-(J22-Pin_3-Pad3) -> GND
- J23 pad 1: GND -> SW5
- J23 pad 2: SW5 -> GND
- J23 pad 3: unconnected-(J23-Pin_3-Pad3) -> GND
- J24 pad 1: GND -> SW6
- J24 pad 2: SW6 -> GND
- J24 pad 3: unconnected-(J24-Pin_3-Pad3) -> GND
- J27 pad 1: GPIO48 -> GND
- J27 pad 2: GPIO47 -> GPIO42
- J27 pad 3: GPIO20 -> GPIO45
- J27 pad 4: GPIO19 -> GPIO46
- J4 pad 1: GND -> VM
- J4 pad 2: VIO -> GND
- J6 pad 1: /SILENTSTEPSTICK Insert n3/EN -> /All TMCs/BothTMCs n1/M2B
- J6 pad 2: SDI -> /All TMCs/BothTMCs n1/M2A
- J6 pad 3: SCK -> /All TMCs/BothTMCs n1/M1A
- J6 pad 4: CS2 -> /All TMCs/BothTMCs n1/M1B
- J7 pad 1: GND -> /All TMCs/BothTMCs n2/M2B
- J7 pad 2: VIO -> /All TMCs/BothTMCs n2/M2A
- J7 pad 3: M1B -> /All TMCs/BothTMCs n2/M1A
- J7 pad 4: M1A -> /All TMCs/BothTMCs n2/M1B
- J8 pad 1: M2B -> /All TMCs/BothTMCs n4/M2B
- J8 pad 2: M2A -> /All TMCs/BothTMCs n4/M2A
- J8 pad 3: M1A -> /All TMCs/BothTMCs n4/M1A
- J8 pad 4: M1B -> /All TMCs/BothTMCs n4/M1B
- J9 pad 1: /SILENTSTEPSTICK Insert2 n5/EN -> /All TMCs/BothTMCs n5/M2B
- J9 pad 2: SDI -> /All TMCs/BothTMCs n5/M2A
- J9 pad 3: SCK -> /All TMCs/BothTMCs n5/M1A
- J9 pad 4: CS3 -> /All TMCs/BothTMCs n5/M1B
Routing:
- net GND: track 0.00 -> 590.7 mm, vias 0 -> 61
- net SDO: track 0.00 -> 332.3 mm, vias 0 -> 7
- net SCK: track 0.00 -> 311.1 mm, vias 0 -> 7
- net SDI: track 0.00 -> 299.3 mm, vias 0 -> 7
- net VM: track 0.00 -> 294.3 mm
- net SW1: track 0.00 -> 157.6 mm
- net SW6: track 0.00 -> 155.7 mm
- net SW5: track 0.00 -> 121.5 mm
- net SW2: track 0.00 -> 115.6 mm
- net VCC: track 0.00 -> 92.8 mm, vias 0 -> 2
- net /All TMCs/DIR6: track 0.00 -> 90.1 mm
- net SW4: track 0.00 -> 89.3 mm
- net /All TMCs/STEP6: track 0.00 -> 83.5 mm
- net SW3: track 0.00 -> 78.8 mm
- net /All TMCs/CS6: track 0.00 -> 71.9 mm
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Other:
- board outline added: 99.1 x 99.1 mm
