File: PCBs/Driver Carrier v1/Driver Carrier v1.kicad_sch (KiCad schematic)
At the start: 12 parts, among them J19 Limit Switch Connector n1, J20 Limit Switch Connector n2, J21 Limit Switch Connector n3, J22 Limit Switch Connector n4, J23 Limit Switch Connector n5, J24 Limit Switch Connector n6, J25 CAN Connector, J26 Controller Reset, J27 Remaining GPIOs, J28 Ground Connectors, J3 Screw_Terminal_01x02, U1 ESP32-S3-DevKitC

Commit message: Continued working on the PCB
Parts:
- removed J28: Ground Connectors, Connector_PinHeader_2.54mm:PinHeader_1x02_P2.54mm_Vertical, symbol Connector:Conn_01x02_Pin
- removed U1: ESP32-S3-DevKitC, Custom_Footprints:ESP32-S3-DEVKITC Female Headers, symbol PCM_Espressif:ESP32-S3-DevKitC
- added J4: Screw_Terminal_01x02, Custom_Footprints:Phoenix_TerminalBlock_1x02_3.5mm_1984617, symbol Connector:Screw_Terminal_01x02
- added U3: ESP32-S3-DEVKITM, Custom_Footprints:ESP32-S3-DEVKITM Female Headers, symbol Custom Symbols:ESP32-S3-DEVKITM_FEMALE_HEADERS
Connections:
- net GPIO48 is gone; now on net GND: J27.1 (Pin_1)
- net CAN_RX: now also U3.27 (RX)
- net CAN_TX: now also U3.28 (TX)
- net CHIP_PU: now also U3.24 (RST)
- net GND: now also J19.2 (Pin_2), J19.3 (Pin_3), J20.2 (Pin_2), J20.3 (Pin_3), J21.2 (Pin_2), J21.3 (Pin_3), J22.2 (Pin_2), J22.3 (Pin_3), J23.2 (Pin_2), J23.3 (Pin_3), J24.2 (Pin_2), J24.3 (Pin_3), J4.2 (Pin_2), U3.22 (GND), U3.23 (GND); no longer J19.1 (Pin_1), J20.1 (Pin_1), J21.1 (Pin_1), J22.1 (Pin_1), J23.1 (Pin_1), J24.1 (Pin_1)
- net SCK: now also U3.32 (GPIO39)
- net SDI: now also U3.31 (GPIO40)
- net SDO: now also U3.30 (GPIO41)
- net SW1: now also J19.1 (Pin_1), U3.15 (GPIO13); no longer J19.2 (Pin_2)
- net SW2: now also J20.1 (Pin_1), U3.16 (GPIO14); no longer J20.2 (Pin_2)
- net SW3: now also J21.1 (Pin_1), U3.17 (GPIO15); no longer J21.2 (Pin_2)
- net SW4: now also J22.1 (Pin_1), U3.18 (GPIO16); no longer J22.2 (Pin_2)
- net SW5: now also J23.1 (Pin_1), U3.19 (GPIO17); no longer J23.2 (Pin_2)
- net SW6: now also J24.1 (Pin_1), U3.20 (GPIO18); no longer J24.2 (Pin_2)
- net VCC: now also U3.21 (5V)
- net VIO: now also U3.1 (3V3)
- net VM: now also J4.1 (Pin_1)
- net GPIO19 renamed GPIO46
- net GPIO46: now also U3.25 (GPIO46)
- net GPIO20 renamed GPIO45
- net GPIO45: now also U3.26 (GPIO45)
- net GPIO47 renamed GPIO42
- net GPIO42: now also U3.29 (GPIO42)
- new net All TMCs/CS1: U3.4 (GPIO2)
- new net All TMCs/CS2: U3.8 (GPIO6)
- new net All TMCs/CS3: U3.12 (GPIO10)
- new net All TMCs/CS4: U3.42 (GPIO19)
- new net All TMCs/CS5: U3.38 (GPIO33)
- new net All TMCs/CS6: U3.34 (GPIO37)
- new net All TMCs/DIR1: U3.6 (GPIO4)
- new net All TMCs/DIR2: U3.10 (GPIO8)
- new net All TMCs/DIR3: U3.14 (GPIO12)
- new net All TMCs/DIR4: U3.44 (GPIO47)
- new net All TMCs/DIR5: U3.40 (GPIO21)
- new net All TMCs/DIR6: U3.36 (GPIO35)
- new net All TMCs/EN1: U3.3 (GPIO1)
- new net All TMCs/EN2: U3.7 (GPIO5)
- new net All TMCs/EN3: U3.11 (GPIO9)
- new net All TMCs/EN4: U3.41 (GPIO20)
- new net All TMCs/EN5: U3.37 (GPIO34)
- new net All TMCs/EN6: U3.33 (GPIO38)
- new net All TMCs/STEP1: U3.5 (GPIO3)
- new net All TMCs/STEP2: U3.9 (GPIO7)
- new net All TMCs/STEP3: U3.13 (GPIO11)
- new net All TMCs/STEP4: U3.43 (GPIO48)
- new net All TMCs/STEP5: U3.39 (GPIO26)
- new net All TMCs/STEP6: U3.35 (GPIO36)
- no-connect marks 6 -> 1
Other:
- removed sheet SILENTSTEPSTICK Insert n1
- removed sheet SILENTSTEPSTICK Insert n2
- removed sheet SILENTSTEPSTICK Insert n3
- removed sheet SILENTSTEPSTICK Insert2 n5
- removed sheet SILENTSTEPSTICK Insert4 n4
- removed sheet SILENTSTEPSTICK Insert5 n6
- added sheet All TMCs (all_tmcs.kicad_sch)
- moved on the sheet: J19, J20, J21, J22, J23, J24, J25, J26, J27, J3
