File: PCBs/Driver Carrier v1/_autosave-Driver Carrier v1.kicad_sch (KiCad schematic)
At the start: 12 parts, among them J10 Limit Switch Connector n4, J11 Limit Switch Connector n5, J12 Limit Switch Connector n6, J13 CAN Connector, J14 Screw_Terminal_01x02, J15 Screw_Terminal_01x02, J16 Controller Reset, J17 Remaining GPIOs, J7 Limit Switch Connector n1, J8 Limit Switch Connector n2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

Commit message: Finished Driver Carrier
Other:
- moved on the sheet: J10, J11, J12, J13, J14, J15, J16, J17, J7, J8, J9
