File: PCBs/Driver Carrier v1/both_tmcs.kicad_sch (KiCad schematic)
At the start: 4 parts, among them J7 Conn_01x04_Pin, U10 SILENTSTEPSTICK TMC5160, U11 SILENTSTEPSTICK TMC2130

Commit message: Finished Driver Carrier
Parts:
- renumbered J7 to J2, U10 to U3, U11 to U4
Changed lines of the file:
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@@
 		(dnp no)
 		(fields_autoplaced yes)
-		(property "Reference" "J7"
+		(property "Reference" "J2"
 			(at 104.14 17.78 90)
 			(effects
@@
 			(project "Driver Carrier v1"
 				(path "/e9233c03-3cf4-4da7-8842-78ed95dae4f3/f38bc85c-7091-4917-a419-8b97603f477b/0dda7cea-57ec-4070-aed0-c52190f2b0cd"
-					(reference "J8")
+					(reference "J4")
 					(unit 1)
 				)
 				(path "/e9233c03-3cf4-4da7-8842-78ed95dae4f3/f38bc85c-7091-4917-a419-8b97603f477b/27e845fa-7a6c-4695-8db7-f6a08065cb82"
+					(reference "J1")
+					(unit 1)
+				)
+				(path "/e9233c03-3cf4-4da7-8842-78ed95dae4f3/f38bc85c-7091-4917-a419-8b97603f477b/60323ed2-c592-4d5f-a3df-90344162b27c"
 					(reference "J6")
 					(unit 1)
 				)
-				(path "/e9233c03-3cf4-4da7-8842-78ed95dae4f3/f38bc85c-7091-4917-a419-8b97603f477b/60323ed2-c592-4d5f-a3df-90344162b27c"
-					(reference "J11")
-					(unit 1)
-				)
 				(path "/e9233c03-3cf4-4da7-8842-78ed95dae4f3/f38bc85c-7091-4917-a419-8b97603f477b/85bfa518-fa29-4b69-81a3-b9a2cd68ceda"
-					(reference "J10")
+					(reference "J3")
 					(unit 1)
 				)
 				(path "/e9233c03-3cf4-4da7-8842-78ed95dae4f3/f38bc85c-7091-4917-a419-8b97603f477b/8a190e82-2a09-4ff3-b645-8ecef9ff4aec"
-					(reference "J7")
+					(reference "J2")
 					(unit 1)
 				)
 				(path "/e9233c03-3cf4-4da7-8842-78ed95dae4f3/f38bc85c-7091-4917-a419-8b97603f477b/9aa1a7ea-d89a-4773-b6a9-df0e8831afe4"
-					(reference "J9")
+					(reference "J5")
 					(unit 1)
 				)
@@
 		(dnp no)
 		(fields_autoplaced yes)
-		(property "Reference" "U10"
+		(property "Reference" "U3"
 			(at 87.63 44.45 0)
 			(effects
@@
 			(project "Driver Carrier v1"
 				(path "/e9233c03-3cf4-4da7-8842-78ed95dae4f3/f38bc85c-7091-4917-a419-8b97603f477b/0dda7cea-57ec-4070-aed0-c52190f2b0cd"
-					(reference "U12")
+					(reference "U7")
 					(unit 1)
 				)
 				(path "/e9233c03-3cf4-4da7-8842-78ed95dae4f3/f38bc85c-7091-4917-a419-8b97603f477b/27e845fa-7a6c-4695-8db7-f6a08065cb82"
-					(reference "U8")
+					(reference "U1")
 					(unit 1)
 				)
 				(path "/e9233c03-3cf4-4da7-8842-78ed95dae4f3/f38bc85c-7091-4917-a419-8b97603f477b/60323ed2-c592-4d5f-a3df-90344162b27c"
-					(reference "U18")
+					(reference "U11")
 					(unit 1)
 				)
 				(path "/e9233c03-3cf4-4da7-8842-78ed95dae4f3/f38bc85c-7091-4917-a419-8b97603f477b/85bfa518-fa29-4b69-81a3-b9a2cd68ceda"
-					(reference "U16")
+					(reference "U5")
 					(unit 1)
 				)
 				(path "/e9233c03-3cf4-4da7-8842-78ed95dae4f3/f38bc85c-7091-4917-a419-8b97603f477b/8a190e82-2a09-4ff3-b645-8ecef9ff4aec"
-					(reference "U10")
+					(reference "U3")
 					(unit 1)
 				)
 				(path "/e9233c03-3cf4-4da7-8842-78ed95dae4f3/f38bc85c-7091-4917-a419-8b97603f477b/9aa1a7ea-d89a-4773-b6a9-df0e8831afe4"
-					(reference "U14")
+					(reference "U9")
 					(unit 1)
 				)
@@
 		(on_board yes)
 		(dnp no)
-		(property "Reference" "U11"
+		(property "Reference" "U4"
 			(at 119.38 44.45 0)
 			(effects
@@
 			(project "Driver Carrier v1"
 				(path "/e9233c03-3cf4-4da7-8842-78ed95dae4f3/f38bc85c-7091-4917-a419-8b97603f477b/0dda7cea-57ec-4070-aed0-c52190f2b0cd"
-					(reference "U13")
+					(reference "U8")
 					(unit 1)
 				)
 				(path "/e9233c03-3cf4-4da7-8842-78ed95dae4f3/f38bc85c-7091-4917-a419-8b97603f477b/27e845fa-7a6c-4695-8db7-f6a08065cb82"
-					(reference "U9")
+					(reference "U2")
 					(unit 1)
 				)
 				(path "/e9233c03-3cf4-4da7-8842-78ed95dae4f3/f38bc85c-7091-4917-a419-8b97603f477b/60323ed2-c592-4d5f-a3df-90344162b27c"
-					(reference "U19")
+					(reference "U12")
 					(unit 1)
 				)
 				(path "/e9233c03-3cf4-4da7-8842-78ed95dae4f3/f38bc85c-7091-4917-a419-8b97603f477b/85bfa518-fa29-4b69-81a3-b9a2cd68ceda"
-					(reference "U17")
+					(reference "U6")
 					(unit 1)
 				)
 				(path "/e9233c03-3cf4-4da7-8842-78ed95dae4f3/f38bc85c-7091-4917-a419-8b97603f477b/8a190e82-2a09-4ff3-b645-8ecef9ff4aec"
-					(reference "U11")
+					(reference "U4")
 					(unit 1)
 				)
 				(path "/e9233c03-3cf4-4da7-8842-78ed95dae4f3/f38bc85c-7091-4917-a419-8b97603f477b/9aa1a7ea-d89a-4773-b6a9-df0e8831afe4"
-					(reference "U15")
-					(unit 1)
-				)
+					(reference "U10")
+					(unit 1)
+				)
